File: PCB/KICAD DESIGN/EnergyMonitor.sch (KiCad schematic (older format))
At the start: 32 parts, among them J1 USB_C_Receptacle_USB2.0, J2 Jack_CTSensor, J3 Screw_Terminal_01x02, J4 Conn_01x04, Q1 2N7002, Q2 2N7002, SW1 SW_Push, SW2 SW_Push, U1 FT232RL, U2 ADS1115IDGS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

Commit message: 2nd release
Connections:
- net CT_SENSOR4: no longer names the net of U3.4 (SENSOR_VP)
- net CT_SENSOR5: no longer names the net of U3.5 (SENSOR_VN)
Changed lines of the file:
@@
 Wire Wire Line
 	2750 3550 3300 3550
-Wire Wire Line
-	11900 2350 12450 2350
-Wire Wire Line
-	11900 2250 12450 2250
-Text Label 12450 2250 2    50   ~ 0
-CT_SENSOR4
-Text Label 12450 2350 2    50   ~ 0
-CT_SENSOR5
 Connection ~ 5250 5150
 $Comp
